Commit message: sync

File: mani_skill/assets/robots/kinova/robotiq_2f_85/robotiq_85.urdf (robot description, URDF)
Before this commit: robot robotiq_arg2f_85_model, 11 links, 10 joints
Joints:
- removed joint finger_joint
- added joint left_outer_knuckle_joint: type revolute, parent robotiq_arg2f_base_link, child left_outer_knuckle, origin xyz=0 -0.0306011 0.054904 rpy=0 0 3.14159265359, axis 1 0 0, limit lower=0 upper=0.8 effort=1000 velocity=2.0
- joint left_inner_finger_joint: mimic joint=finger_joint multiplier=-1 offset=0 -> joint=left_outer_knuckle_joint multiplier=-1 offset=0
- joint left_inner_knuckle_joint: mimic joint=finger_joint multiplier=1 offset=0 -> joint=left_outer_knuckle_joint multiplier=1 offset=0
- joint right_inner_finger_joint: mimic joint=finger_joint multiplier=-1 offset=0 -> joint=left_outer_knuckle_joint multiplier=-1 offset=0
- joint right_inner_knuckle_joint: mimic joint=finger_joint multiplier=1 offset=0 -> joint=left_outer_knuckle_joint multiplier=1 offset=0
- joint right_outer_knuckle_joint: mimic joint=finger_joint multiplier=1 offset=0 -> joint=left_outer_knuckle_joint multiplier=1 offset=0
