Commit message: fix kinova+robotiq2f85; fix video record; update demo_side_grasp; update init pose of panda and kinova

File: mani_skill/assets/robots/kinova/gen3_dof7_robotiq_2f_140.urdf (robot description, URDF)
Before this commit: robot gen3_robotiq_2f_140, 24 links, 23 joints
Joints:
- joint right_outer_knuckle_joint: axis 1 0 0 -> -1 0 0; limit lower=-0.725 upper=0 effort=1000 velocity=2.0 -> lower=0 upper=0.725 effort=1000 velocity=2.0
